Commit message: fix URDF Linux通信 Mini9

File: src/models/MINI/mini_model/urdf/mini.urdf (robot description, URDF)
Before this commit: robot mini, 16 links, 15 joints
Links:
- removed link RealSence_B
- removed link RealSence_F
Joints:
- removed joint RealSence_B_Joint
- removed joint RealSence_F_Joint
